File: RFBoardLayoutGen0_v03.3JK2.sch (EAGLE design)
At the start: 78 parts

Commit message: Backup commit
Parts:
- added U$11, U$12, U$13, U$14: LP-FILTER/VARACTOR/0402, LPFilter:LP-FILTER/VARACTOR/0402
Connections:
- removed net $1234567254654: E$2.25, LP$1.GND, LP$10.GND, LP$11.GND, LP$12.GND, LP$13.GND, LP$14.GND, LP$15.GND, LP$16.GND, LP$17.GND, LP$18.GND, LP$19.GND, LP$2.GND, LP$20.GND, LP$21.GND, LP$22.GND, LP$23.GND, LP$24.GND, LP$3.GND, LP$4.GND, LP$5.GND, LP$6.GND, LP$7.GND, LP$8.GND, LP$9.GND, S$1.GND@1, S$2.GND@1, S$3.GND@1, S$4.GND@1, S$5.GND@1, S$6.GND@1, S$7.GND@1, U$1.25, U$1.26
- net GND: now also E$2.25, LP$1.GND, LP$10.GND, LP$11.GND, LP$12.GND, LP$13.GND, LP$14.GND, LP$15.GND, LP$16.GND, LP$17.GND, LP$18.GND, LP$19.GND, LP$2.GND, LP$20.GND, LP$21.GND, LP$22.GND, LP$23.GND, LP$24.GND, LP$3.GND, LP$4.GND, LP$5.GND, LP$6.GND, LP$7.GND, LP$8.GND, LP$9.GND, S$1.GND@1, S$2.GND@1, S$3.GND@1, S$4.GND@1, S$5.GND@1, S$6.GND@1, S$7.GND@1, U$1.25, U$1.26
- net N$10: now also U$14.1
- net N$11: now also U$13.1
- net N$2: now also U$12.1
- net N$9: now also U$11.1
