File: RFBoardLayoutGen0_v03.3JK2.brd (EAGLE design)
At the start: 76.9 x 40.1 mm, 83 parts

Commit message: DRC error solving
Parts:
- removed E$30: (no value), PADS:SMD0.8-0,5
- moved U$10 0.07 mm to (7.41, 8.19)
- moved U$9 0.07 mm to (7.37, -8.18)
Routing:
- net GND: track 8.25 -> 10.0 mm, vias 505 -> 507
- net D$10: track 70.5 -> 72.2 mm
- net D$15: track 81.3 -> 82.8 mm
- net D$14: track 64.3 -> 65.5 mm
- net D$18: track 58.0 -> 57.0 mm
- net D$13: track 63.3 -> 64.1 mm
- net D$12: track 70.3 -> 71.1 mm
- net D$11: track 73.9 -> 74.7 mm
- net D$16: track 69.8 -> 70.5 mm
- net D$5: track 77.2 -> 77.7 mm
- net N$9: vias 0 -> 2
- net N$2: vias 0 -> 2
- net N$11: vias 0 -> 2
- net N$10: vias 0 -> 2
Other:
- board text added: "G1"
- board text added: "G2"
- board text added: "G3"
- board text added: "G4"
- board text added: "G5"
- board text added: "G6"
