File: RFBoardLayoutGen0_v03.3JK2.brd (EAGLE design)
At the start: 76.9 x 40.1 mm, 82 parts

Commit message: Seems finished
Routing:
- net D$8: track 78.3 -> 84.7 mm
- net D$7: track 74.2 -> 80.2 mm
- net D$9: track 80.0 -> 85.7 mm
- net D$15: track 82.8 -> 86.4 mm
- net D$14: track 65.5 -> 67.6 mm
- net D$13: track 64.1 -> 66.2 mm
- net D$4: track 66.8 -> 68.9 mm
- net D$5: track 77.7 -> 79.7 mm
- net D$12: track 71.1 -> 69.3 mm
- net GND: track 10.0 -> 11.8 mm, vias 507 -> 543
- net D$6: track 73.1 -> 71.7 mm
- net D$10: track 72.2 -> 71.1 mm
- net D$17: track 57.1 -> 58.1 mm
- net D$18: track 57.0 -> 58.0 mm
- net D$3: track 64.0 -> 64.6 mm
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