File: RFBoardLayoutGen0_v03.4.brd (EAGLE design)
At the start: 76.9 x 40.1 mm, 82 parts

Commit message: DRC solved
Parts:
- moved U$14 3.47 mm to (-1.01, 0.52)
- moved U$13 3.04 mm to (1.51, 0.77)
Routing:
- net D$7: track 74.1 -> 80.2 mm
- net D$9: track 80.0 -> 85.7 mm
- net D$8: track 80.8 -> 84.7 mm
- net D$15: track 84.5 -> 86.4 mm
- net D$6: track 72.9 -> 71.7 mm
- net D$5: track 79.7 -> 78.9 mm
- net GND: vias 523 -> 543

Commit message: v3.4 prefinished
Parts:
- added U$17, U$18: LP-FILTER/CAPACITOR/0402, LPFilter:LP-FILTER/CAPACITOR/0402
- added U$19, U$20, U$21, U$22: LP-FILTER/RESISTOR/0402, LPFilter:LP-FILTER/CAPACITOR/0402
- U$15, U$16: value LP-FILTER/CAPACITOR/0603 -> LP-FILTER/CAPACITOR/0402; device LPFilter:LP-FILTER/CAPACITOR/0603_BOTTOM -> LPFilter:LP-FILTER/CAPACITOR/0402
- moved U$15 5.09 mm to (-2.12, 3.50), turned to 180 degrees
- moved U$16 5.09 mm to (-2.12, -3.50), turned to 0 degrees
- moved U$14 3.62 mm to (-0.75, 4.12), turned to 90 degrees
- moved U$13 3.44 mm to (0.75, 4.12), turned to 90 degrees
- moved U$11 1.82 mm to (-0.76, -4.14), turned to 270 degrees
- moved U$12 1.82 mm to (0.76, -4.14), turned to 270 degrees
Connections:
- new net N$29: U$13.IN, U$17.IN, U$19.OUT, U$22.OUT
- new net N$35: U$12.IN, U$18.OUT, U$20.OUT, U$21.IN
- new net N$36: U$14.IN, U$15.IN, U$19.IN
- new net N$37: U$11.IN, U$16.OUT, U$20.IN
- net D$15: now also U$21.OUT; no longer U$11.OUT, U$12.OUT, U$16.OUT
- net D$5: now also U$22.IN; no longer U$13.OUT, U$14.OUT, U$15.OUT
- net GND: now also U$11.OUT, U$12.OUT, U$13.OUT, U$14.OUT; no longer U$15.IN, U$16.IN
- net N$10: now also U$15.OUT; no longer U$14.IN
- net N$11: now also U$17.OUT; no longer U$13.IN
- net N$2: now also U$18.IN; no longer U$12.IN
- net N$9: now also U$16.IN; no longer U$11.IN
Routing:
- net GND: track 11.8 -> 26.8 mm
- net D$5: track 78.9 -> 72.6 mm
- net D$15: track 86.4 -> 80.5 mm
- net N$35: track 0.00 -> 4.60 mm
- net N$29: track 0.00 -> 4.58 mm
- net N$37: track 0.00 -> 1.75 mm
- net N$36: track 0.00 -> 1.73 mm
